File: OutsideFoilSniffer.kicad_sch (KiCad schematic)
At the start: 40 parts, among them J1 Black, J2 Red, J3 Signal, J4 Conn_01x15_Male, J5 Conn_01x15_Male, K1 SANYOU_SRD_Form_C, Q1 BC547, Q2 2N3904

Commit message: Modified size to fit PCBWay prototype size 100x80 mm for cheap price
Parts:
- C1: footprint Capacitor_THT:C_Rect_L7.0mm_W2.5mm_P5.00mm -> Capacitor_THT:C_Rect_L10.0mm_W3.0mm_P7.50mm_MKS4
- C5: footprint Capacitor_THT:C_Rect_L7.0mm_W2.5mm_P5.00mm -> Capacitor_THT:C_Rect_L13.0mm_W4.0mm_P10.00mm_FKS3_FKP3_MKS4
Changed lines of the file:
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@@
       (effects (font (size 1.27 1.27)) (justify left))
     )
-    (property "Footprint" "Capacitor_THT:C_Rect_L7.0mm_W2.5mm_P5.00mm" (id 2) (at 46.355 167.3098 0)
+    (property "Footprint" "Capacitor_THT:C_Rect_L13.0mm_W4.0mm_P10.00mm_FKS3_FKP3_MKS4" (id 2) (at 46.355 167.3098 0)
       (effects (font (size 1.27 1.27)) hide)
     )
@@
     (property "Reference" "C1" (id 0) (at 73.025 152.2562 90))
     (property "Value" "0.01uf" (id 1) (at 73.025 154.7931 90))
-    (property "Footprint" "Capacitor_THT:C_Rect_L7.0mm_W2.5mm_P5.00mm" (id 2) (at 69.215 159.0802 0)
+    (property "Footprint" "Capacitor_THT:C_Rect_L10.0mm_W3.0mm_P7.50mm_MKS4" (id 2) (at 69.215 159.0802 0)
       (effects (font (size 1.27 1.27)) hide)
     )
@@
     )
     (path "/c6c6f9b2-9f87-4788-b46d-8e510305084d"
-      (reference "C1") (unit 1) (value "0.01uf") (footprint "Capacitor_THT:C_Rect_L7.0mm_W2.5mm_P5.00mm")
+      (reference "C1") (unit 1) (value "0.01uf") (footprint "Capacitor_THT:C_Rect_L10.0mm_W3.0mm_P7.50mm_MKS4")
     )
     (path "/4d71057e-54cb-4a1b-a5c4-4601df070c6b"
@@
     )
     (path "/8f363f0e-d267-4359-9c3d-fb4f788e37e4"
-      (reference "C5") (unit 1) (value "0.15uf") (footprint "Capacitor_THT:C_Rect_L7.0mm_W2.5mm_P5.00mm")
+      (reference "C5") (unit 1) (value "0.15uf") (footprint "Capacitor_THT:C_Rect_L13.0mm_W4.0mm_P10.00mm_FKS3_FKP3_MKS4")
     )
     (path "/16f6c8c5-9c37-4ffd-8143-a0c82434fde0"

Commit message: Added sniffer code modified for my design. Code needs serious cleanup
Parts:
- D1, D2: footprint Diode_THT:D_DO-35_SOD27_P7.62mm_Horizontal -> Diode_THT:D_DO-35_SOD27_P10.16mm_Horizontal
- R1: value R -> 470K
- R10, R9: value R -> 220
- R2: value R -> 4K7
- R3: value R -> 1K
- R4, R8: value R -> 10K
- R5: value R -> 100K
- R6, R7: value R -> 470
Changed lines of the file:
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@@
     (property "Reference" "D1" (id 0) (at 84.455 167.005 0))
     (property "Value" "1N34A" (id 1) (at 79.375 167.005 0))
-    (property "Footprint" "Diode_THT:D_DO-35_SOD27_P7.62mm_Horizontal" (id 2) (at 77.47 167.005 0)
+    (property "Footprint" "Diode_THT:D_DO-35_SOD27_P10.16mm_Horizontal" (id 2) (at 77.47 167.005 0)
       (effects (font (size 1.27 1.27)) hide)
     )
@@
     (in_bom yes) (on_board yes)
     (property "Reference" "R10" (id 0) (at 227.838 97.155 90))
-    (property "Value" "R" (id 1) (at 229.87 97.155 90))
+    (property "Value" "220" (id 1) (at 229.87 97.155 90))
     (property "Footprint" "Resistor_THT:R_Axial_DIN0207_L6.3mm_D2.5mm_P10.16mm_Horizontal" (id 2) (at 231.648 97.155 90)
       (effects (font (size 1.27 1.27)) hide)
@@
     (property "Reference" "D2" (id 0) (at 90.805 153.1452 0))
     (property "Value" "1N34A" (id 1) (at 90.805 155.6821 0))
-    (property "Footprint" "Diode_THT:D_DO-35_SOD27_P7.62mm_Horizontal" (id 2) (at 90.805 153.67 0)
+    (property "Footprint" "Diode_THT:D_DO-35_SOD27_P10.16mm_Horizontal" (id 2) (at 90.805 153.67 0)
       (effects (font (size 1.27 1.27)) hide)
     )
@@
     (in_bom yes) (on_board yes)
     (property "Reference" "R5" (id 0) (at 111.887 167.005 90))
-    (property "Value" "R" (id 1) (at 109.855 167.005 90))
+    (property "Value" "100K" (id 1) (at 109.855 167.005 90))
     (property "Footprint" "Resistor_THT:R_Axial_DIN0207_L6.3mm_D2.5mm_P10.16mm_Horizontal" (id 2) (at 108.077 167.005 90)
       (effects (font (size 1.27 1.27)) hide)
@@
     (in_bom yes) (on_board yes)
     (property "Reference" "R9" (id 0) (at 242.062 97.155 90))
-    (property "Value" "R" (id 1) (at 240.03 97.155 90))
+    (property "Value" "220" (id 1) (at 240.03 97.155 90))
     (property "Footprint" "Resistor_THT:R_Axial_DIN0207_L6.3mm_D2.5mm_P10.16mm_Horizontal" (id 2) (at 238.252 97.155 90)
       (effects (font (size 1.27 1.27)) hide)
@@
       (effects (font (size 1.27 1.27)) (justify right))
     )
-    (property "Value" "R" (id 1) (at 43.053 76.6322 0)
+    (property "Value" "10K" (id 1) (at 43.053 76.6322 0)
       (effects (font (size 1.27 1.27)) (justify right))
     )
@@
     (in_bom yes) (on_board yes)
     (property "Reference" "R7" (id 0) (at 70.485 35.687 90))
-    (property "Value" "R" (id 1) (at 70.485 33.655 90))
+    (property "Value" "470" (id 1) (at 70.485 33.655 90))
     (property "Footprint" "Resistor_THT:R_Axial_DIN0207_L6.3mm_D2.5mm_P10.16mm_Horizontal" (id 2) (at 70.485 31.877 90)
       (effects (font (size 1.27 1.27)) hide)
@@
       (effects (font (size 1.27 1.27)) (justify left))
     )
-    (property "Value" "R" (id 1) (at 68.7828 40.513 0)
+    (property "Value" "470" (id 1) (at 68.7828 40.513 0)
       (effects (font (size 1.27 1.27)) (justify left))
     )
@@
       (effects (font (size 1.27 1.27)) (justify left))
     )
-    (property "Value" "R" (id 1) (at 53.213 147.7522 0)
+    (property "Value" "4K7" (id 1) (at 53.213 147.7522 0)
       (effects (font (size 1.27 1.27)) (justify left))
     )
@@
     (in_bom yes) (on_board yes)
     (property "Reference" "R8" (id 0) (at 85.852 111.76 90))
-    (property "Value" "R" (id 1) (at 83.82 111.76 90))
+    (property "Value" "10K" (id 1) (at 83.82 111.76 90))
     (property "Footprint" "Resistor_THT:R_Axial_DIN0207_L6.3mm_D2.5mm_P10.16mm_Horizontal" (id 2) (at 82.042 111.76 90)
       (effects (font (size 1.27 1.27)) hide)
@@
     (in_bom yes) (on_board yes)
     (property "Reference" "R3" (id 0) (at 47.625 66.548 90))
-    (property "Value" "R" (id 1) (at 47.625 68.58 90))
+    (property "Value" "1K" (id 1) (at 47.625 68.58 90))
     (property "Footprint" "Resistor_THT:R_Axial_DIN0207_L6.3mm_D2.5mm_P10.16mm_Horizontal" (id 2) (at 47.625 70.358 90)
       (effects (font (size 1.27 1.27)) hide)
@@
     (in_bom yes) (on_board yes)
     (property "Reference" "R1" (id 0) (at 53.467 159.385 90))
-    (property "Value" "R" (id 1) (at 51.435 159.385 90))
+    (property "Value" "470K" (id 1) (at 51.435 159.385 90))
     (property "Footprint" "Resistor_THT:R_Axial_DIN0207_L6.3mm_D2.5mm_P10.16mm_Horizontal" (id 2) (at 49.657 159.385 90)
       (effects (font (size 1.27 1.27)) hide)
@@
     )
     (path "/16f6c8c5-9c37-4ffd-8143-a0c82434fde0"
-      (reference "D1") (unit 1) (value "1N34A") (footprint "Diode_THT:D_DO-35_SOD27_P7.62mm_Horizontal")
+      (reference "D1") (unit 1) (value "1N34A") (footprint "Diode_THT:D_DO-35_SOD27_P10.16mm_Horizontal")
     )
     (path "/4583d84f-bda5-4c0b-92c3-e7ece4146667"
-      (reference "D2") (unit 1) (value "1N34A") (footprint "Diode_THT:D_DO-35_SOD27_P7.62mm_Horizontal")
+      (reference "D2") (unit 1) (value "1N34A") (footprint "Diode_THT:D_DO-35_SOD27_P10.16mm_Horizontal")
     )
     (path "/43e5c75b-c249-4518-9877-e80dacf98940"
@@
     )
     (path "/f08dd9aa-50c7-4a88-af5a-e184364f2582"
-      (reference "R1") (unit 1) (value "R") (footprint "Resistor_THT:R_Axial_DIN0207_L6.3mm_D2.5mm_P10.16mm_Horizontal")
+      (reference "R1") (unit 1) (value "470K") (footprint "Resistor_THT:R_Axial_DIN0207_L6.3mm_D2.5mm_P10.16mm_Horizontal")
     )
     (path "/ae956af1-fa60-4cba-bddb-39bd126fcbf0"
-      (reference "R2") (unit 1) (value "R") (footprint "Resistor_THT:R_Axial_DIN0207_L6.3mm_D2.5mm_P10.16mm_Horizontal")
+      (reference "R2") (unit 1) (value "4K7") (footprint "Resistor_THT:R_Axial_DIN0207_L6.3mm_D2.5mm_P10.16mm_Horizontal")
     )
     (path "/db4ea57f-14a2-4d0a-8c6f-739496e34c0c"
-      (reference "R3") (unit 1) (value "R") (footprint "Resistor_THT:R_Axial_DIN0207_L6.3mm_D2.5mm_P10.16mm_Horizontal")
+      (reference "R3") (unit 1) (value "1K") (footprint "Resistor_THT:R_Axial_DIN0207_L6.3mm_D2.5mm_P10.16mm_Horizontal")
     )
     (path "/902befea-9daa-4b4e-a709-e3aa02ab039f"
-      (reference "R4") (unit 1) (value "R") (footprint "Resistor_THT:R_Axial_DIN0207_L6.3mm_D2.5mm_P10.16mm_Horizontal")
+      (reference "R4") (unit 1) (value "10K") (footprint "Resistor_THT:R_Axial_DIN0207_L6.3mm_D2.5mm_P10.16mm_Horizontal")
     )
     (path "/4aadcca9-0618-4454-beda-336d23708a05"
-      (reference "R5") (unit 1) (value "R") (footprint "Resistor_THT:R_Axial_DIN0207_L6.3mm_D2.5mm_P10.16mm_Horizontal")
+      (reference "R5") (unit 1) (value "100K") (footprint "Resistor_THT:R_Axial_DIN0207_L6.3mm_D2.5mm_P10.16mm_Horizontal")
     )
     (path "/a51fba43-7598-4cf8-81ac-5ba6abf5ccda"
-      (reference "R6") (unit 1) (value "R") (footprint "Resistor_THT:R_Axial_DIN0207_L6.3mm_D2.5mm_P10.16mm_Horizontal")
+      (reference "R6") (unit 1) (value "470") (footprint "Resistor_THT:R_Axial_DIN0207_L6.3mm_D2.5mm_P10.16mm_Horizontal")
     )
     (path "/92c4f962-e6df-406e-9173-2bb2a1cb9744"
-      (reference "R7") (unit 1) (value "R") (footprint "Resistor_THT:R_Axial_DIN0207_L6.3mm_D2.5mm_P10.16mm_Horizontal")
+      (reference "R7") (unit 1) (value "470") (footprint "Resistor_THT:R_Axial_DIN0207_L6.3mm_D2.5mm_P10.16mm_Horizontal")
     )
     (path "/bf9285db-8992-4772-8655-2a606cd52b20"
-      (reference "R8") (unit 1) (value "R") (footprint "Resistor_THT:R_Axial_DIN0207_L6.3mm_D2.5mm_P10.16mm_Horizontal")
+      (reference "R8") (unit 1) (value "10K") (footprint "Resistor_THT:R_Axial_DIN0207_L6.3mm_D2.5mm_P10.16mm_Horizontal")
     )
     (path "/4bd5a113-2059-43da-b1ca-7e5cbf46b4a9"
-      (reference "R9") (unit 1) (value "R") (footprint "Resistor_THT:R_Axial_DIN0207_L6.3mm_D2.5mm_P10.16mm_Horizontal")
+      (reference "R9") (unit 1) (value "220") (footprint "Resistor_THT:R_Axial_DIN0207_L6.3mm_D2.5mm_P10.16mm_Horizontal")
     )
     (path "/3281ee27-b62e-4931-8b2c-d61043a1c301"
-      (reference "R10") (unit 1) (value "R") (footprint "Resistor_THT:R_Axial_DIN0207_L6.3mm_D2.5mm_P10.16mm_Horizontal")
-    )
-  )
+      (reference "R10") (unit 1) (value "220") (footprint "Resistor_THT:R_Axial_DIN0207_L6.3mm_D2.5mm_P10.16mm_Horizontal")
+    )
+  )

Commit message: minor changes
Parts:
- Q1, Q2: footprint Package_TO_SOT_THT:TO-92_Inline -> Package_TO_SOT_THT:TO-92_Inline_Wide
Changed lines of the file:
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@@
       (effects (font (size 1.27 1.27)) (justify left))
     )
-    (property "Footprint" "Package_TO_SOT_THT:TO-92_Inline" (id 2) (at 28.575 70.485 0)
+    (property "Footprint" "Package_TO_SOT_THT:TO-92_Inline_Wide" (id 2) (at 28.575 70.485 0)
       (effects (font (size 1.27 1.27) italic) (justify left) hide)
     )
@@
       (effects (font (size 1.27 1.27)) (justify left))
     )
-    (property "Footprint" "Package_TO_SOT_THT:TO-92_Inline" (id 2) (at 66.675 170.18 0)
+    (property "Footprint" "Package_TO_SOT_THT:TO-92_Inline_Wide" (id 2) (at 66.675 170.18 0)
       (effects (font (size 1.27 1.27) italic) (justify left) hide)
     )
@@
     )
     (path "/7e7de603-30a0-40ff-9e65-870b69f11c12"
-      (reference "Q1") (unit 1) (value "BC547") (footprint "Package_TO_SOT_THT:TO-92_Inline")
+      (reference "Q1") (unit 1) (value "BC547") (footprint "Package_TO_SOT_THT:TO-92_Inline_Wide")
     )
     (path "/3eb55c5a-2336-4e6d-9970-410cd2e1b309"
-      (reference "Q2") (unit 1) (value "2N3904") (footprint "Package_TO_SOT_THT:TO-92_Inline")
+      (reference "Q2") (unit 1) (value "2N3904") (footprint "Package_TO_SOT_THT:TO-92_Inline_Wide")
     )
     (path "/f08dd9aa-50c7-4a88-af5a-e184364f2582"
